File: Multi-LED_JT_V2.sch (KiCad schematic (older format))
At the start: 11 parts, among them Q1 BC817-25

Commit message: remove switch
Parts:
- removed S1: SPDT, lib_fp:SPDT_OS102011MA1QN1, symbol SPDT
Connections:
- wire segments 27 -> 26
Changed lines of the file:
@@
-$EndComp
-$Comp
-L SPDT S1
-U 1 1 59ED576C
-P 3650 3600
-F 0 "S1" H 3650 3400 60  0000 C CNN
-F 1 "SPDT" H 3650 3850 60  0000 C CNN
-F 2 "lib_fp:SPDT_OS102011MA1QN1" H 3650 3600 60  0001 C CNN
-F 3 "" H 3650 3600 60  0000 C CNN
-F 4 "C&K" H 3650 3600 60  0001 C CNN "Manufacture"
-F 5 "OS102011MA1QN1" H 3650 3600 60  0001 C CNN "Mfg Part Number"
-F 6 "THT" H 3650 3600 60  0001 C CNN "Package"
-F 7 "SWITCH SLIDE SPDT 100MA 12V" H 3650 3600 60  0001 C CNN "Description"
-	1    3650 3600
-	1    0    0    -1
 $EndComp
 $Comp
@@
 $EndComp
 Wire Wire Line
-	2850 4250 2850 3600
-Wire Wire Line
-	2850 3600 3400 3600
-Wire Wire Line
-	3750 3500 4350 3500
-Wire Wire Line
 	4350 3800 4200 3800
 Wire Wire Line
@@
 	7300 4750 7300 4700
 Connection ~ 7300 4700
+Wire Wire Line
+	2850 3500 4350 3500
+Wire Wire Line
+	2850 3500 2850 4250
 $EndSCHEMATC

Commit message: D1 Annode not connected
Connections:
- wire segments 26 -> 38
Changed lines of the file:
@@
 	5750 4200 5750 3500
 Wire Wire Line
-	5150 3500 8050 3500
+	5150 3500 5750 3500
+Wire Wire Line
+	5750 3500 6550 3500
+Wire Wire Line
+	6550 3500 6850 3500
+Wire Wire Line
+	6850 3500 7150 3500
+Wire Wire Line
+	7150 3500 7450 3500
+Wire Wire Line
+	7450 3500 7750 3500
+Wire Wire Line
+	7750 3500 8050 3500
 $Comp
 L GND #PWR01
@@
 Connection ~ 6850 3500
 Wire Wire Line
-	6550 4200 6550 3500
+	6550 4250 6550 3500
 Connection ~ 6550 3500
 Wire Wire Line
 	6550 4550 6550 4700
 Wire Wire Line
-	6550 4700 8050 4700
+	6550 4700 6850 4700
+Wire Wire Line
+	6850 4700 7150 4700
+Wire Wire Line
+	7150 4700 7300 4700
+Wire Wire Line
+	7300 4700 7450 4700
+Wire Wire Line
+	7450 4700 7750 4700
+Wire Wire Line
+	7750 4700 8050 4700
 Wire Wire Line
 	8050 4700 8050 4550
@@
 Connection ~ 7300 4700
 Wire Wire Line
-	2850 3500 4350 3500
+	2850 3500 4200 3500
+Wire Wire Line
+	4200 3500 4350 3500
 Wire Wire Line
 	2850 3500 2850 4250

Commit message: D1 anode not connected
Changed lines of the file:
@@
 	5750 4200 5750 3500
 Wire Wire Line
-	5150 3500 5750 3500
-Wire Wire Line
-	5750 3500 6550 3500
-Wire Wire Line
-	6550 3500 6850 3500
-Wire Wire Line
-	6850 3500 7150 3500
-Wire Wire Line
-	7150 3500 7450 3500
-Wire Wire Line
-	7450 3500 7750 3500
-Wire Wire Line
-	7750 3500 8050 3500
+	5150 3500 8050 3500
 $Comp
 L GND #PWR01
@@
 	6550 4550 6550 4700
 Wire Wire Line
-	6550 4700 6850 4700
-Wire Wire Line
-	6850 4700 7150 4700
-Wire Wire Line
-	7150 4700 7300 4700
-Wire Wire Line
-	7300 4700 7450 4700
-Wire Wire Line
-	7450 4700 7750 4700
-Wire Wire Line
-	7750 4700 8050 4700
+	6550 4700 8050 4700
 Wire Wire Line
 	8050 4700 8050 4550
@@
 Connection ~ 7300 4700
 Wire Wire Line
-	2850 3500 4200 3500
-Wire Wire Line
-	4200 3500 4350 3500
+	2850 3500 4350 3500
 Wire Wire Line
 	2850 3500 2850 4250

Commit message: add DPDT JS202011JAQN switch
Parts:
- added SW?: SW_DPDT, symbol SW_DPDT_x2
Connections:
- net GND: now also SW?.2 (B); no longer BT1.2 (-)
- new net: BT1.2 (-), SW?.3 (C)
Changed lines of the file:
@@
 L GND #PWR02
 U 1 1 59EFDBF0
-P 2850 4600
-F 0 "#PWR02" H 2850 4350 50  0001 C CNN
-F 1 "GND" H 2850 4450 50  0000 C CNN
-F 2 "" H 2850 4600 50  0001 C CNN
-F 3 "" H 2850 4600 50  0001 C CNN
-	1    2850 4600
+P 2750 5050
+F 0 "#PWR02" H 2750 4800 50  0001 C CNN
+F 1 "GND" H 2750 4900 50  0000 C CNN
+F 2 "" H 2750 5050 50  0001 C CNN
+F 3 "" H 2750 5050 50  0001 C CNN
+	1    2750 5050
 	1    0    0    -1
 $EndComp
@@
 Wire Wire Line
 	2850 3500 2850 4250
+$Comp
+L SW_DPDT_x2 SW?
+U 1 1 5A1C120C
+P 2750 4800
+F 0 "SW?" H 2750 4970 50  0000 C CNN
+F 1 "SW_DPDT" H 2750 4600 50  0000 C CNN
+F 2 "" H 2750 4800 50  0001 C CNN
+F 3 "" H 2750 4800 50  0001 C CNN
+F 4 "CK" H 2750 4800 60  0001 C CNN "Manufacture"
+F 5 "JS202011JAQN" H 2750 4800 60  0001 C CNN "Mfg Part Number"
+F 6 "SMD" H 2750 4800 60  0001 C CNN "Package"
+F 7 "SWITCH SLIDE DPDT 300MA 6V" H 2750 4800 60  0001 C CNN "Description"
+	1    2750 4800
+	0    -1   -1   0
+$EndComp
+Wire Wire Line
+	2750 5050 2750 5000
 $EndSCHEMATC
